File: hardware/fk-weather.kicad_pcb (KiCad board)
At the start: 2 copper layers, 28.7 x 87.4 mm, 99 parts, among them J1 MICRO-USB, J2 CONN_01X03, J3 CONN_01X06, J5 Conn_01x01, J6 CONN-HDR-2x5, J7 Conn_01x01, J8 Conn_01x01, J9 Conn_01x01, M1 MOUNT_HOLE, M2 MOUNT_HOLE, M3 MOUNT_HOLE, M4 MOUNT_HOLE, Q1 2N7002LT1G, Q2 2N7002LT1G, Q3 2N7002LT1G, Q4 2N7002LT1G, SW1 SPNO, U1 ATSAMD21G18A-AU, U101 TSL2591, U102 MPL3115A2, U103 BNO055, U104 SHT31, U2 MCP1700T-XXX2E, U3 MAX4466, U4 S25FL1xxK0XM, Y1 FC-135, Y101 FC-135

Commit message: Fix version number.
Other:
- board text added: "v0.5"
- board text removed: "v0.4"
Changed lines of the file:
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@@
     (links 208)
     (no_connects 0)
-    (area 125.718499 67.742999 154.578121 155.274081)
+    (area 106.352905 47.75 165.914286 159.377948)
     (thickness 1.6)
     (drawings 27)
@@
     (effects (font (size 1 1) (thickness 0.25)))
   )
-  (gr_text v0.4 (at 147.574 154.178) (layer F.SilkS)
+  (gr_text v0.5 (at 147.574 154.178) (layer F.SilkS)
     (effects (font (size 1.2 1.2) (thickness 0.2)))
   )

Commit message: Adding another breakout for the MIC to attach a header to for probing.
Parts:
- added J4: Conn_01x02, Socket_Strips:Socket_Strip_Straight_2x01_Pitch2.54mm, F.Cu at (135.3, 70.7)
Routing:
- net /AGND: track 18.7 -> 29.6 mm
- net 3V3: track 267.8 -> 274.9 mm
- net Net-(C15-Pad2): track 9.38 -> 16.0 mm
Other:
- board text added: "A1"
- board text added: "MIC"
Changed lines of the file:
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@@
 (kicad_pcb (version 4) (host pcbnew 4.0.7-e2-6376~58~ubuntu16.04.1)
   (general
-    (links 208)
-    (no_connects 0)
-    (area 106.352905 47.75 165.914286 159.377948)
+    (links 210)
+    (no_connects 43)
+    (area 125.718499 67.742999 154.578121 155.274081)
     (thickness 1.6)
-    (drawings 27)
-    (tracks 785)
+    (drawings 32)
+    (tracks 795)
     (zones 0)
-    (modules 99)
+    (modules 100)
     (nets 97)
   )
@@
     )
   )
+  (module Socket_Strips:Socket_Strip_Straight_2x01_Pitch2.54mm (layer F.Cu)
+    (at 135.2804 70.7136)
+    (descr "Through hole straight socket strip, 2x01, 2.54mm pitch, double rows")
+    (tags "Through hole socket strip THT 2x01 2.54mm double row")
+    (fp_text reference J4 (at -1.27 -2.33) (layer F.SilkS) hide
+      (effects (font (size 1 1) (thickness 0.15)))
+    )
+    (fp_text value Conn_01x02 (at -1.27 2.33) (layer F.Fab)
+      (effects (font (size 1 1) (thickness 0.15)))
+    )
+    (fp_line (start -3.81 -1.27) (end -3.81 1.27) (layer F.Fab) (width 0.1))
+    (fp_line (start -3.81 1.27) (end 1.27 1.27) (layer F.Fab) (width 0.1))
+    (fp_line (start 1.27 1.27) (end 1.27 -1.27) (layer F.Fab) (width 0.1))
+    (fp_line (start 1.27 -1.27) (end -3.81 -1.27) (layer F.Fab) (width 0.1))
+    (fp_line (start 1.33 1.27) (end 1.33 1.33) (layer F.SilkS) (width 0.12))
+    (fp_line (start 1.33 1.33) (end -3.87 1.33) (layer F.SilkS) (width 0.12))
+    (fp_line (start -3.87 1.33) (end -3.87 -1.33) (layer F.SilkS) (width 0.12))
+    (fp_line (start -3.87 -1.33) (end -1.27 -1.33) (layer F.SilkS) (width 0.12))
+    (fp_line (start -1.27 -1.33) (end -1.27 1.27) (layer F.SilkS) (width 0.12))
+    (fp_line (start -1.27 1.27) (end 1.33 1.27) (layer F.SilkS) (width 0.12))
+    (fp_line (start 1.33 0) (end 1.33 -1.33) (layer F.SilkS) (width 0.12))
+    (fp_line (start 1.33 -1.33) (end 0.06 -1.33) (layer F.SilkS) (width 0.12))
+    (fp_line (start -4.35 -1.8) (end -4.35 1.8) (layer F.CrtYd) (width 0.05))
+    (fp_line (start -4.35 1.8) (end 1.8 1.8) (layer F.CrtYd) (width 0.05))
+    (fp_line (start 1.8 1.8) (end 1.8 -1.8) (layer F.CrtYd) (width 0.05))
+    (fp_line (start 1.8 -1.8) (end -4.35 -1.8) (layer F.CrtYd) (width 0.05))
+    (fp_text user %R (at -1.27 -2.33) (layer F.Fab)
+      (effects (font (size 1 1) (thickness 0.15)))
+    )
+    (pad 1 thru_hole rect (at 0 0) (size 1.7 1.7) (drill 1) (layers *.Cu *.Mask)
+      (net 77 "Net-(C15-Pad2)"))
+    (pad 2 thru_hole oval (at -2.54 0) (size 1.7 1.7) (drill 1) (layers *.Cu *.Mask)
+      (net 75 /AGND))
+    (model ${KISYS3DMOD}/Socket_Strips.3dshapes/Socket_Strip_Straight_2x01_Pitch2.54mm.wrl
+      (at (xyz -0.05 0 0))
+      (scale (xyz 1 1 1))
+      (rotate (xyz 0 0 270))
+    )
+  )
+  (gr_text MIC (at 139.192 80.7466) (layer F.SilkS)
+    (effects (font (size 0.8 0.8) (thickness 0.2)))
+  )
+  (gr_text MIC (at 134.0358 73.1266) (layer F.SilkS)
+    (effects (font (size 0.8 0.8) (thickness 0.2)))
+  )
+  (gr_text 3V3 (at 139.2682 73.1774) (layer F.SilkS)
+    (effects (font (size 0.8 0.8) (thickness 0.2)))
+  )
+  (gr_text A1 (at 144.3228 73.152) (layer F.SilkS)
+    (effects (font (size 0.8 0.8) (thickness 0.2)))
+  )
+  (gr_text GND (at 141.7574 73.152) (layer F.SilkS)
+    (effects (font (size 0.8 0.8) (thickness 0.2)))
+  )
   (gr_arc (start 153.74112 154.43708) (end 154.50312 154.43708) (angle 90) (layer Edge.Cuts) (width 0.15))
   (gr_arc (start 126.56312 154.43708) (end 126.52756 155.19908) (angle 87.32813541) (layer Edge.Cuts) (width 0.15))
@@
   (segment (start 140.945949 97.306051) (end 140.945949 98.121317) (width 0.254) (layer F.Cu) (net 3))
   (segment (start 140.945949 98.121317) (end 139.821883 99.245383) (width 0.254) (layer F.Cu) (net 3))
+  (segment (start 130.2004 68.834) (end 130.2004 76.4032) (width 0.254) (layer B.Cu) (net 4))
+  (segment (start 130.2004 76.4032) (end 129.2352 77.3684) (width 0.254) (layer B.Cu) (net 4))
+  (segment (start 130.6322 68.4022) (end 130.2004 68.834) (width 0.254) (layer B.Cu) (net 4))
+  (segment (start 138.0862 68.4022) (end 130.6322 68.4022) (width 0.254) (layer B.Cu) (net 4))
+  (segment (start 139.319 70.739) (end 139.319 69.635) (width 0.254) (layer B.Cu) (net 4))
+  (segment (start 139.319 69.635) (end 138.0862 68.4022) (width 0.254) (layer B.Cu) (net 4))
   (segment (start 139.352 88.5825) (end 139.352 89.8525) (width 0.254) (layer F.Cu) (net 4))
   (segment (start 131.445 90.49) (end 131.445 87.9221) (width 0.254) (layer F.Cu) (net 4))
@@
   (segment (start 136.093755 108.717584) (end 135.144339 109.667) (width 0.254) (layer F.Cu) (net 4))
   (segment (start 135.144339 109.667) (end 133.858 109.667) (width 0.254) (layer F.Cu) (net 4))
-  (segment (start 139.319 70.739) (end 135.8646 70.739) (width 0.254) (layer B.Cu) (net 4))
-  (segment (start 135.8646 70.739) (end 129.2352 77.3684) (width 0.254) (layer B.Cu) (net 4))
   (segment (start 146.558 88.9) (end 143.3195 88.9) (width 0.254) (layer F.Cu) (net 4))
   (segment (start 143.3195 88.9) (end 141.605 87.1855) (width 0.254) (layer F.Cu) (net 4))
@@
   (segment (start 149.421 73.8935) (end 148.717 73.8935) (width 0.254) (layer F.Cu) (net 74))
   (segment (start 147.066 73.8935) (end 148.717 73.8935) (width 0.254) (layer F.Cu) (net 74))
+  (segment (start 137.2108 77.4183) (end 137.2108 75.184) (width 0.254) (layer F.Cu) (net 75))
+  (segment (start 137.2108 75.184) (end 132.7404 70.7136) (width 0.254) (layer F.Cu) (net 75))
+  (segment (start 139.192 78.2955) (end 138.088 78.2955) (width 0.254) (layer F.Cu) (net 75))
+  (segment (start 138.088 78.2955) (end 137.2108 77.4183) (width 0.254) (layer F.Cu) (net 75))
   (segment (start 142.56 77.7875) (end 140.804 77.7875) (width 0.254) (layer F.Cu) (net 75))
   (segment (start 140.804 77.7875) (end 140.296 78.2955) (width 0.254) (layer F.Cu) (net 75))
@@
   (segment (start 141.859 76.6875) (end 141.859 74.9275) (width 0.254) (layer F.Cu) (net 76))
   (segment (start 141.859 74.9275) (end 141.798 74.8665) (width 0.254) (layer F.Cu) (net 76))
+  (segment (start 139.192 75.7555) (end 135.2804 71.8439) (width 0.254) (layer F.Cu) (net 77))
+  (segment (start 135.2804 71.8439) (end 135.2804 70.7136) (width 0.254) (layer F.Cu) (net 77))
   (segment (start 139.192 75.7555) (end 140.735401 74.212099) (width 0.254) (layer F.Cu) (net 77))
   (segment (start 140.735401 74.212099) (end 142.818599 74.212099) (width 0.254) (layer F.Cu) (net 77))
