File: hardware/sensor-board/fk-weather-sensors.sch (KiCad schematic (older format))
At the start: 9 parts, among them J1 CONN_01X06, U1 MPL3115A2, U2 TSL2591, U3 SHT31

Commit message: Change header orien. Plot.
Connections:
- net labels removed: 5V0
- wire segments 44 -> 42
Changed lines of the file:
@@
-$EndComp
-$Comp
-L 5V0 #PWR2
-U 1 1 5A446545
-P 5550 5450
-F 0 "#PWR2" H 5550 5300 50  0001 C CNN
-F 1 "5V0" H 5550 5590 50  0000 C CNN
-F 2 "" H 5550 5450 60  0000 C CNN
-F 3 "" H 5550 5450 60  0000 C CNN
-	1    5550 5450
-	1    0    0    -1
 $EndComp
 $Comp
@@
 	1    0    0    -1
 $EndComp
-Text Label 5750 5350 0    50   ~ 0
+Text Label 5750 5250 0    50   ~ 0
 SDA
-Text Label 5750 5250 0    50   ~ 0
+Text Label 5750 5150 0    50   ~ 0
 SCL
 Text Label 8250 5350 2    50   ~ 0
@@
 NoConn ~ 8400 5450
 NoConn ~ 7800 1700
-NoConn ~ 5650 5150
-Wire Wire Line
-	5750 5250 6000 5250
-Wire Wire Line
-	5750 5350 6000 5350
-Wire Wire Line
-	5650 5150 6000 5150
 Wire Wire Line
 	5750 4950 6000 4950
@@
 	5550 5050 5550 5000
 Wire Wire Line
-	6000 5450 5550 5450
-Wire Wire Line
 	7550 1800 7800 1800
 Wire Wire Line
@@
 Text Notes 2150 800  0    118  ~ 24
 MPL3115A2 (PRESSURE/HUMIDITY)
+NoConn ~ 6000 5450
+Wire Wire Line
+	5750 5150 6000 5150
+Wire Wire Line
+	6000 5250 5750 5250
 $EndSCHEMATC

Commit message: Fix TSL2591 footprint.
Parts:
- U2: footprint Housings_DFN_QFN:DFN-6-1EP_2x2mm_Pitch0.65mm -> conservify:TSL2591
Changed lines of the file:
@@
 $EndDescr
 $Comp
-L 3V3 #PWR1
+L 3V3 #PWR01
 U 1 1 5A4464F2
 P 5550 5000
-F 0 "#PWR1" H 5550 4850 50  0001 C CNN
+F 0 "#PWR01" H 5550 4850 50  0001 C CNN
 F 1 "3V3" H 5550 5140 50  0000 C CNN
 F 2 "" H 5550 5000 60  0000 C CNN
@@
 $EndComp
 $Comp
-L GND #PWR3
+L GND #PWR02
 U 1 1 5A4464F3
 P 5750 4800
-F 0 "#PWR3" H 5750 4550 50  0001 C CNN
+F 0 "#PWR02" H 5750 4550 50  0001 C CNN
 F 1 "GND" H 5750 4650 50  0001 C CNN
 F 2 "" H 5750 4800 60  0000 C CNN
@@
 $EndComp
 $Comp
-L GND #PWR5
+L GND #PWR03
 U 1 1 5A4464F5
 P 4800 2800
-F 0 "#PWR5" H 4800 2550 50  0001 C CNN
+F 0 "#PWR03" H 4800 2550 50  0001 C CNN
 F 1 "GND" H 4800 2650 50  0001 C CNN
 F 2 "" H 4800 2800 60  0000 C CNN
@@
 F 0 "U2" H 9050 5350 60  0000 C CNN
 F 1 "TSL2591" H 9050 5450 60  0000 C CNN
-F 2 "Housings_DFN_QFN:DFN-6-1EP_2x2mm_Pitch0.65mm" H 9050 5350 60  0001 C CNN
+F 2 "conservify:TSL2591" H 9050 5350 60  0001 C CNN
 F 3 "" H 9050 5350 60  0001 C CNN
 F 4 "0" H 9050 5450 50  0001 C CNN "price"
@@
 $EndComp
 $Comp
-L 3V3 #PWR4
+L 3V3 #PWR04
 U 1 1 5A4464FA
 P 4800 1700
-F 0 "#PWR4" H 4800 1550 50  0001 C CNN
+F 0 "#PWR04" H 4800 1550 50  0001 C CNN
 F 1 "3V3" H 4800 1840 50  0000 C CNN
 F 2 "" H 4800 1700 60  0000 C CNN
@@
 $EndComp
 $Comp
-L GND #PWR7
+L GND #PWR05
 U 1 1 5A4464FB
 P 10550 5850
-F 0 "#PWR7" H 10550 5600 50  0001 C CNN
+F 0 "#PWR05" H 10550 5600 50  0001 C CNN
 F 1 "GND" H 10550 5700 50  0001 C CNN
 F 2 "" H 10550 5850 60  0000 C CNN
@@
 $EndComp
 $Comp
-L 3V3 #PWR6
+L 3V3 #PWR06
 U 1 1 5A4464FC
 P 10550 5200
-F 0 "#PWR6" H 10550 5050 50  0001 C CNN
+F 0 "#PWR06" H 10550 5050 50  0001 C CNN
 F 1 "3V3" H 10550 5340 50  0000 C CNN
 F 2 "" H 10550 5200 60  0000 C CNN
@@
 $EndComp
 $Comp
-L GND #PWR10
+L GND #PWR07
 U 1 1 5A446500
 P 10050 1950
-F 0 "#PWR10" H 10050 1700 50  0001 C CNN
+F 0 "#PWR07" H 10050 1700 50  0001 C CNN
 F 1 "GND" H 10050 1800 50  0001 C CNN
 F 2 "" H 10050 1950 60  0000 C CNN
@@
 $EndComp
 $Comp
-L 3V3 #PWR9
+L 3V3 #PWR08
 U 1 1 5A446501
 P 10050 1400
-F 0 "#PWR9" H 10050 1250 50  0001 C CNN
+F 0 "#PWR08" H 10050 1250 50  0001 C CNN
 F 1 "3V3" H 10050 1540 50  0000 C CNN
 F 2 "" H 10050 1400 60  0000 C CNN
@@
 $EndComp
 $Comp
-L GND #PWR8
+L GND #PWR09
 U 1 1 5A446546
 P 7550 1950
-F 0 "#PWR8" H 7550 1700 50  0001 C CNN
+F 0 "#PWR09" H 7550 1700 50  0001 C CNN
 F 1 "GND" H 7550 1800 50  0001 C CNN
 F 2 "" H 7550 1950 60  0000 C CNN

Commit message: Add RTC. Molex connector cleanup. Add RGB LED.Fix diode footprints.
Parts:
- removed J1: CONN_01X06, Socket_Strips:Socket_Strip_Straight_1x06_Pitch2.54mm, symbol CONN_01X06
- added J1: CONN_01x04, conservify:Molex_CLIK-Mate_502382-0470_1x04_P1.25mm_Vertical, symbol CONN_01x04
- C1, C2, C3, C4, C5: footprint Capacitors_SMD:C_0603_HandSoldering -> conservify:CAP-0603
Connections:
- no-connect marks 5 -> 4
Changed lines of the file:
@@
 EESchema Schematic File Version 2
-LIBS:power
-LIBS:device
-LIBS:switches
-LIBS:relays
-LIBS:motors
-LIBS:transistors
-LIBS:conn
-LIBS:linear
-LIBS:regul
-LIBS:74xx
-LIBS:cmos4000
-LIBS:adc-dac
-LIBS:memory
-LIBS:xilinx
-LIBS:microcontrollers
-LIBS:dsp
-LIBS:microchip
-LIBS:analog_switches
-LIBS:motorola
-LIBS:texas
-LIBS:intel
-LIBS:audio
-LIBS:interface
-LIBS:digital-audio
-LIBS:philips
-LIBS:display
-LIBS:cypress
-LIBS:siliconi
-LIBS:opto
-LIBS:atmel
-LIBS:contrib
-LIBS:valves
+LIBS:conservify
 LIBS:fk-weather-sensors-cache
 EELAYER 25 0
@@
 $EndDescr
 $Comp
-L 3V3 #PWR01
+L 3V3 #PWR4
 U 1 1 5A4464F2
+P 5750 4800
+F 0 "#PWR4" H 5750 4650 50  0001 C CNN
+F 1 "3V3" H 5750 4940 50  0000 C CNN
+F 2 "" H 5750 4800 60  0000 C CNN
+F 3 "" H 5750 4800 60  0000 C CNN
+	1    5750 4800
+	1    0    0    -1
+$EndComp
+$Comp
+L GND #PWR3
+U 1 1 5A4464F3
 P 5550 5000
-F 0 "#PWR01" H 5550 4850 50  0001 C CNN
-F 1 "3V3" H 5550 5140 50  0000 C CNN
+F 0 "#PWR3" H 5550 4750 50  0001 C CNN
+F 1 "GND" H 5550 4850 50  0001 C CNN
 F 2 "" H 5550 5000 60  0000 C CNN
 F 3 "" H 5550 5000 60  0000 C CNN
 	1    5550 5000
-	1    0    0    -1
-$EndComp
-$Comp
-L GND #PWR02
-U 1 1 5A4464F3
-P 5750 4800
-F 0 "#PWR02" H 5750 4550 50  0001 C CNN
-F 1 "GND" H 5750 4650 50  0001 C CNN
-F 2 "" H 5750 4800 60  0000 C CNN
-F 3 "" H 5750 4800 60  0000 C CNN
-	1    5750 4800
 	-1   0    0    1
 $EndComp
@@
 $EndComp
 $Comp
-L GND #PWR03
+L GND #PWR2
 U 1 1 5A4464F5
 P 4800 2800
-F 0 "#PWR03" H 4800 2550 50  0001 C CNN
+F 0 "#PWR2" H 4800 2550 50  0001 C CNN
 F 1 "GND" H 4800 2650 50  0001 C CNN
 F 2 "" H 4800 2800 60  0000 C CNN
@@
 F 0 "C1" V 4200 2150 50  0000 L CNN
 F 1 "100nF" V 4500 2100 50  0000 L CNN
-F 2 "Capacitors_SMD:C_0603_HandSoldering" H 4350 2000 30  0001 C CNN
+F 2 "conservify:CAP-0603" H 4350 2000 30  0001 C CNN
 F 3 "" H 4350 2200 60  0000 C CNN
 F 4 "0" H 4200 2250 50  0001 C CNN "price"
@@
 F 0 "C2" V 4650 2150 50  0000 L CNN
 F 1 "100nF" V 4950 2100 50  0000 L CNN
-F 2 "Capacitors_SMD:C_0603_HandSoldering" H 4800 2000 30  0001 C CNN
+F 2 "conservify:CAP-0603" H 4800 2000 30  0001 C CNN
 F 3 "" H 4800 2200 60  0000 C CNN
 F 4 "0" H 4650 2250 50  0001 C CNN "price"
@@
 F 0 "C4" V 5100 2150 50  0000 L CNN
 F 1 "10uF" V 5400 2100 50  0000 L CNN
-F 2 "Capacitors_SMD:C_0603_HandSoldering" H 5250 2000 30  0001 C CNN
+F 2 "conservify:CAP-0603" H 5250 2000 30  0001 C CNN
 F 3 "" H 5250 2200 60  0000 C CNN
 F 4 "0" H 5100 2250 50  0001 C CNN "price"
@@
 $EndComp
 $Comp
-L 3V3 #PWR04
+L 3V3 #PWR1
 U 1 1 5A4464FA
 P 4800 1700
-F 0 "#PWR04" H 4800 1550 50  0001 C CNN
+F 0 "#PWR1" H 4800 1550 50  0001 C CNN
 F 1 "3V3" H 4800 1840 50  0000 C CNN
 F 2 "" H 4800 1700 60  0000 C CNN
@@
 $EndComp
 $Comp
-L GND #PWR05
+L GND #PWR9
 U 1 1 5A4464FB
 P 10550 5850
-F 0 "#PWR05" H 10550 5600 50  0001 C CNN
+F 0 "#PWR9" H 10550 5600 50  0001 C CNN
 F 1 "GND" H 10550 5700 50  0001 C CNN
 F 2 "" H 10550 5850 60  0000 C CNN
@@
 $EndComp
 $Comp
-L 3V3 #PWR06
+L 3V3 #PWR8
 U 1 1 5A4464FC
 P 10550 5200
-F 0 "#PWR06" H 10550 5050 50  0001 C CNN
+F 0 "#PWR8" H 10550 5050 50  0001 C CNN
 F 1 "3V3" H 10550 5340 50  0000 C CNN
 F 2 "" H 10550 5200 60  0000 C CNN
@@
 F 0 "C3" V 10400 5450 50  0000 L CNN
 F 1 "1uF" V 10700 5450 50  0000 L CNN
-F 2 "Capacitors_SMD:C_0603_HandSoldering" H 10550 5300 30  0001 C CNN
+F 2 "conservify:CAP-0603" H 10550 5300 30  0001 C CNN
 F 3 "" H 10550 5500 60  0000 C CNN
 F 4 "0" H 10400 5550 50  0001 C CNN "price"
@@
 F 0 "C5" V 9900 1600 50  0000 L CNN
 F 1 "100nF" V 10200 1550 50  0000 L CNN
-F 2 "Capacitors_SMD:C_0603_HandSoldering" H 10050 1450 30  0001 C CNN
+F 2 "conservify:CAP-0603" H 10050 1450 30  0001 C CNN
 F 3 "" H 10050 1650 60  0000 C CNN
 F 4 "0" H 9900 1700 50  0001 C CNN "price"
@@
 $EndComp
 $Comp
-L GND #PWR07
+L GND #PWR7
 U 1 1 5A446500
 P 10050 1950
-F 0 "#PWR07" H 10050 1700 50  0001 C CNN
+F 0 "#PWR7" H 10050 1700 50  0001 C CNN
 F 1 "GND" H 10050 1800 50  0001 C CNN
 F 2 "" H 10050 1950 60  0000 C CNN
@@
 $EndComp
 $Comp
-L 3V3 #PWR08
+L 3V3 #PWR6
 U 1 1 5A446501
 P 10050 1400
-F 0 "#PWR08" H 10050 1250 50  0001 C CNN
+F 0 "#PWR6" H 10050 1250 50  0001 C CNN
 F 1 "3V3" H 10050 1540 50  0000 C CNN
 F 2 "" H 10050 1400 60  0000 C CNN
@@
 $EndComp
 $Comp
-L CONN_01X06 J1
-U 1 1 5A446544
-P 6200 5200
-F 0 "J1" H 6200 5550 50  0000 C CNN
-F 1 "CONN_01X06" V 6300 5200 50  0000 C CNN
-F 2 "Socket_Strips:Socket_Strip_Straight_1x06_Pitch2.54mm" H 6200 5200 50  0001 C CNN
-F 3 "" H 6200 5200 50  0001 C CNN
-F 4 "0" H 6200 5650 50  0001 C CNN "price"
-	1    6200 5200
-	1    0    0    -1
-$EndComp
-$Comp
-L GND #PWR09
+L GND #PWR5
 U 1 1 5A446546
 P 7550 1950
-F 0 "#PWR09" H 7550 1700 50  0001 C CNN
+F 0 "#PWR5" H 7550 1700 50  0001 C CNN
 F 1 "GND" H 7550 1800 50  0001 C CNN
 F 2 "" H 7550 1950 60  0000 C CNN
@@
 Text Notes 2150 800  0    118  ~ 24
 MPL3115A2 (PRESSURE/HUMIDITY)
-NoConn ~ 6000 5450
 Wire Wire Line
 	5750 5150 6000 5150
 Wire Wire Line
 	6000 5250 5750 5250
+$Comp
+L CONN_01x04 J1
+U 1 1 5B584D44
+P 6200 5050
+F 0 "J1" H 6200 5250 50  0000 C CNN
+F 1 "CONN_01x04" H 6200 4750 50  0000 C CNN
+F 2 "conservify:Molex_CLIK-Mate_502382-0470_1x04_P1.25mm_Vertical" H 6200 5050 50  0001 C CNN
+F 3 "" H 6200 5050 50  0001 C CNN
+	1    6200 5050
+	1    0    0    -1
+$EndComp
 $EndSCHEMATC
