File: hardware/sensor-board/fk-weather-sensors.sch (KiCad schematic (older format))
At the start: 9 parts, among them J1 CONN_01x04, U1 MPL3115A2, U2 TSL2591, U3 SHT31

Commit message: Part updates.
Parts:
- C1, C2, C5: Critical (none) -> (none); MFN (none) -> Murata Electronics; MFP (none) -> GRM188R71H104KA93D; Notes (none) -> (none); Package (none) -> (none); Source (none) -> ANY; Subsystem (none) -> (none)
- C3: Critical (none) -> (none); MFN (none) -> Taiyo Yuden; MFP (none) -> UMK107BJ105KA-T; Notes (none) -> (none); Package (none) -> (none); Source (none) -> ANY; Subsystem (none) -> (none)
- C4: Critical (none) -> (none); MFN (none) -> Taiyo Yuden; MFP (none) -> LMK107BBJ106KALT; Notes (none) -> (none); Package (none) -> (none); Source (none) -> ANY; Subsystem (none) -> (none); spn1 81-GRM188R60J106ME47 -> 963-LMK107BBJ106KALT
- J1: Critical (none) -> (none); MFN (none) -> (none); MFP (none) -> (none); Notes (none) -> (none); Package (none) -> (none); SPN1 (none) -> (none); Source (none) -> ANY; Subsystem (none) -> (none); Supplier1 (none) -> (none)
- U1: Critical (none) -> (none); MFN (none) -> NXP / Freescale; MFP (none) -> MPL3115A2; Notes (none) -> (none); Package (none) -> (none); Source (none) -> ANY; Subsystem (none) -> (none)
- U2: Critical (none) -> (none); MFN (none) -> AMS; MFP (none) -> TSL25911FN; Notes (none) -> (none); Package (none) -> (none); Source (none) -> ANY; Subsystem (none) -> (none)
- U3: Critical (none) -> (none); MFN (none) -> Sensirion; MFP (none) -> SHT31-DIS-B; Notes (none) -> (none); Package (none) -> (none); Source (none) -> ANY; Subsystem (none) -> (none)

Commit message: Fix rescued stuff and clear DRC problems.
Parts:
- C1, C2, C3, C4, C5: symbol fk-weather-sensors-rescue:CAPACITOR-CERAMIC -> conservify:CAPACITOR_CERAMIC
Connections:
- wire segments 52 -> 54

Commit message: Consistency in part values
Parts:
- J1: MFN (none) -> Molex; MFP (none) -> 502382-0470; SPN1 (none) -> WM4781CT-ND; Supplier1 (none) -> digikey
