File: hardware/module-board/fk-weather.sch (KiCad schematic (older format))
At the start: 71 parts, among them J1 MICRO-USB, J10 Conn_01x06, J11 Conn_01x06, J2 Conn_01x05, J3 CONN_01x03_SERIAL, J4 Conn_01x04, J5 Conn_01x02, J6 CONN_02x05_SWD, J7 Conn_01x05, M1 MOUNT_HOLE, M2 MOUNT_HOLE, M3 MOUNT_HOLE, M4 MOUNT_HOLE, Q4 2N7002LT1G, SW1 SPNO, U1 ATSAMD21G18A-AU, U2 MCP1700T-XXX2E, U3 TPS2051B, U4 S25FL1xxK0XM, U5 SK6812, U6 PCF8523, Y1 FC-135, Y2 FC-135

Commit message: Consistent part values across our schematics.
Parts:
- C14: value 4.7uF 10V X5R -> 4.7uF
- C5: value 1uF 10V X5R -> 1uF
- R8: value 100k -> 100K
- U2: value MCP1700T-XXX2E -> MCP1700T-3302E/MB
- U4: value S25FL1xxK0XM -> S25FL116K0XMFI041

Commit message: Part updates.
Parts:
- BT1, D10, D11, D6, D7, D8, D9, J10, J11, J5, M1, M2, M3, M4, U3: Critical (none) -> (none); MFN (none) -> (none); MFP (none) -> (none); Notes (none) -> (none); Package (none) -> (none); SPN1 (none) -> (none); Source (none) -> ANY; Subsystem (none) -> (none); Supplier1 (none) -> (none)
- C1, C2: Critical (none) -> (none); MFN (none) -> AVX; MFP (none) -> 06035A180JAT2A; Notes (none) -> (none); Package (none) -> (none); Source (none) -> ANY; Subsystem (none) -> (none)
- C10: Critical (none) -> (none); MFN (none) -> KEMET; MFP (none) -> C0603C472K9RACTU; Notes (none) -> (none); Package (none) -> (none); Source (none) -> ANY; Subsystem (none) -> (none)
- C11, C12: Critical (none) -> (none); MFN (none) -> Taiyo Yuden; MFP (none) -> UMK107BJ105KA-T; Notes (none) -> (none); Package (none) -> (none); Source (none) -> ANY; Subsystem (none) -> (none)
- C13, C15, C18, C3, C4, C6, C7, C8: Critical (none) -> (none); MFN (none) -> Murata Electronics; MFP (none) -> GRM188R71H104KA93D; Notes (none) -> (none); Package (none) -> (none); Source (none) -> ANY; Subsystem (none) -> (none)
- C14, C9: Critical (none) -> (none); MFN (none) -> AVX; MFP (none) -> 0603ZD475MAT2A; Notes (none) -> (none); Package (none) -> (none); Source (none) -> ANY; Subsystem (none) -> (none)
- C16: Critical (none) -> (none); MFN (none) -> Taiyo Yuden; MFP (none) -> LMK107BBJ106KALT; Notes (none) -> (none); Package (none) -> (none); SPN1 (none) -> 963-LMK107BBJ106KALT; Source (none) -> ANY; Subsystem (none) -> (none)
- C17, C19: Critical (none) -> (none); MFN (none) -> AVX; MFP (none) -> 0603YC103K4T2A; Notes (none) -> (none); Package (none) -> (none); SPN1 (none) -> 581-0603YC103K4T2A; Source (none) -> ANY; Subsystem (none) -> (none)
- C5: Critical (none) -> (none); MFN (none) -> Taiyo Yuden; MFP (none) -> UMK107BJ105KA-T; Notes (none) -> (none); Package (none) -> (none); Source (none) -> ANY; Subsystem (none) -> (none); spn1 581-0603YD105K -> 963-UMK107BJ105KA-T
- D4: Critical (none) -> (none); MFN (none) -> Nexperia; MFP (none) -> PRTR5V0U2X,215; Notes (none) -> (none); Package (none) -> (none); Source (none) -> ANY; Subsystem (none) -> (none)
- D5: Critical (none) -> (none); MFN (none) -> Lite-On; MFP (none) -> LTST-C190KFKT; Notes (none) -> (none); Package (none) -> (none); Source (none) -> ANY; Subsystem (none) -> (none)
- F1: Critical (none) -> (none); MFN (none) -> Bourns; MFP (none) -> MF-PSMF050X-2; Notes (none) -> (none); Package (none) -> (none); Source (none) -> ANY; Subsystem (none) -> (none)
- J1: Critical (none) -> (none); MFN (none) -> Hirose Connector; MFP (none) -> ZX62D-B-5PA8(30); Notes (none) -> (none); Package (none) -> (none); Source (none) -> ANY; Subsystem (none) -> (none); Supplier1 (none) -> mouser
- J2, J7: Critical (none) -> (none); MFN (none) -> Molex; MFP (none) -> 502382-0570; Notes (none) -> (none); Package (none) -> (none); SPN1 (none) -> 538-502382-0570; Source (none) -> ANY; Subsystem (none) -> (none); Supplier1 (none) -> mouser
- J3: Critical (none) -> (none); MFN (none) -> Molex; MFP (none) -> 502382-0370; Notes (none) -> (none); Package (none) -> (none); SPN1 (none) -> 538-502382-0370; Source (none) -> ANY; Subsystem (none) -> (none); Supplier1 (none) -> mouser
- J4: value Conn_01x04 -> CONN_01x04; Critical (none) -> (none); MFN (none) -> (none); MFP (none) -> (none); Notes (none) -> (none); Package (none) -> (none); SPN1 (none) -> (none); Source (none) -> ANY; Subsystem (none) -> (none); Supplier1 (none) -> (none)
- J6: Critical (none) -> (none); MFN (none) -> Amphenol FCI; MFP (none) -> 20021121-00010C4LF; Notes (none) -> (none); Package (none) -> (none); SPN1 (none) -> 649-202112100010C4LF; Source (none) -> ANY; Subsystem (none) -> (none); Supplier1 (none) -> mouser
- L1, L2: Critical (none) -> (none); MFN (none) -> Murata Electronics; MFP (none) -> BLM18KG221SN1D; Notes (none) -> (none); Package (none) -> (none); Source (none) -> ANY; Subsystem (none) -> (none)
- Q4: Critical (none) -> (none); MFN (none) -> ON Semiconductor; MFP (none) -> 2N7002LT1G; Notes (none) -> (none); Package (none) -> (none); Source (none) -> ANY; Subsystem (none) -> (none)
- R1: Critical (none) -> (none); MFN (none) -> (none); MFP (none) -> (none); Notes (none) -> (none); Package (none) -> (none); SPN1 (none) -> 603-RC0603FR-07330RL; Source (none) -> ANY; Subsystem (none) -> (none)
- R10: Critical (none) -> (none); MFN (none) -> Yageo; MFP (none) -> RC0603FR-071ML; Notes (none) -> (none); Package (none) -> (none); Source (none) -> ANY; Subsystem (none) -> (none)
- R11, R4: Critical (none) -> (none); MFN (none) -> Yageo; MFP (none) -> RC0603FR-0710KL; Notes (none) -> (none); Package (none) -> (none); Source (none) -> ANY; Subsystem (none) -> (none)
- R17, R22, R23, R30, R31, R32, R33: Critical (none) -> (none); MFN (none) -> (none); MFP (none) -> (none); Notes (none) -> (none); Package (none) -> (none); Source (none) -> ANY; Subsystem (none) -> (none)
- R2, R9: Critical (none) -> (none); MFN (none) -> Yageo; MFP (none) -> RC0603FR-07330RL; Notes (none) -> (none); Package (none) -> (none); Source (none) -> ANY; Subsystem (none) -> (none)
- R34, R6, R7: Critical (none) -> (none); MFN (none) -> Yageo; MFP (none) -> AF0603JR-074K7L; Notes (none) -> (none); Package (none) -> (none); Source (none) -> ANY; Subsystem (none) -> (none)
- R8: Critical (none) -> (none); MFN (none) -> Yageo; MFP (none) -> RC0603FR-07100KL; Notes (none) -> (none); Package (none) -> (none); Source (none) -> ANY; Subsystem (none) -> (none)
- SW1: Critical (none) -> (none); MFN (none) -> Wurth Electronics; MFP (none) -> 434331045822; Notes (none) -> (none); Package (none) -> (none); Source (none) -> ANY; Subsystem (none) -> (none); Supplier1 (none) -> digikey
- U1: Critical (none) -> (none); MFN (none) -> Microchip Technology / Atmel; MFP (none) -> ATSAMD21G18A-AU; Notes (none) -> (none); Package (none) -> (none); Source (none) -> ANY; Subsystem (none) -> (none)
- U2: Critical (none) -> (none); MFN (none) -> Microchip Technology; MFP (none) -> MCP1700T-3302E/MB; Notes (none) -> (none); Package (none) -> (none); Source (none) -> ANY; Subsystem (none) -> (none)
- U4: Critical (none) -> (none); MFN (none) -> Cypress Semiconductor; MFP (none) -> S25FL116K0XMFI041; Notes (none) -> (none); Package (none) -> (none); Source (none) -> ANY; Subsystem (none) -> (none); Supplier1 (none) -> mouser
- U5: Critical (none) -> (none); MFN (none) -> Adafruit; MFP (none) -> 1655; Notes (none) -> (none); Package (none) -> (none); SPN1 (none) -> 1528-1104-ND; Source (none) -> ANY; Subsystem (none) -> (none); Supplier1 (none) -> digikey
- U6: Critical (none) -> (none); MFN (none) -> NXP Semiconductors; MFP (none) -> PCF8523T/1,118; Notes (none) -> (none); Package (none) -> (none); SPN1 (none) -> 771-PCF8523T/1118; Source (none) -> ANY; Subsystem (none) -> (none); Supplier1 (none) -> mouser
- Y1, Y2: Critical (none) -> (none); MFN (none) -> Epson Timing; MFP (none) -> FC-135 32.7680KA-A3; Notes (none) -> (none); Package (none) -> (none); Source (none) -> ANY; Subsystem (none) -> (none)

Commit message: Fix SK6812 and cleanup signal naming.
Connections:
- net labels added: A1_WIND_DIR, D10_WIND_SPEED, D5_FLASH_CS, D6_RAIN, D8_PERIPH_EN
- net labels removed: FLASH_CS, PERIPH_EN, RAIN, WIND_DIR, WIND_SPEED

Commit message: Fix rescued stuff and clear DRC problems.
Parts:
- C1, C10, C11, C12, C13, C14, C15, C16, C17, C18, C19, C2, C3, C4, C5, C6, C7, C8, C9: symbol fk-weather-rescue:CAPACITOR-CERAMIC -> conservify:CAPACITOR_CERAMIC
- D5: symbol fk-weather-rescue:LED-SINGLE -> conservify:LED_SINGLE
- J1: symbol fk-weather-rescue:MICRO-USB -> conservify:MICRO_USB
- J10, J11: symbol fk-weather-rescue:Conn_01x06 -> conservify:CONN_01x06
- J2, J7: symbol fk-weather-rescue:Conn_01x05 -> conservify:CONN_01x05
- J4: symbol fk-weather-rescue:Conn_01x04 -> conservify:CONN_01x04
- J5: symbol fk-weather-rescue:Conn_01x02 -> conservify:CONN_01x02
- Q4: symbol fk-weather-rescue:MOSFET-N -> conservify:MOSFET_N
- SW1: symbol fk-weather-rescue:TACT-SWITCH_2Pins -> conservify:SWITCH_CONN_02
- U1: symbol fk-weather-rescue:ATSAMD21G18A-AU -> conservify:ATSAMD21G18A_AU
Connections:
- net labels removed: AREF
- wire segments 286 -> 287
- no-connect marks 9 -> 29
Changed lines of the file:
@@
 $EndDescr
 $Comp
-L fk-weather-rescue:TACT-SWITCH_2Pins SW1
+L conservify:SWITCH_CONN_02 SW1
 U 1 1 56091122
 P 3900 2050
@@
 $EndComp
 $Comp
-L fk-weather-rescue:CAPACITOR-CERAMIC C2
+L conservify:CAPACITOR_CERAMIC C2
 U 1 1 560BC402
 P 2950 1800
@@
 $EndComp
 $Comp
-L fk-weather-rescue:CAPACITOR-CERAMIC C1
+L conservify:CAPACITOR_CERAMIC C1
 U 1 1 560BC473
 P 2250 1800
@@
 $EndComp
 $Comp
-L fk-weather-rescue:CAPACITOR-CERAMIC C3
+L conservify:CAPACITOR_CERAMIC C3
 U 1 1 560C00D4
 P 5350 2300
@@
 $EndComp
 $Comp
-L fk-weather-rescue:CAPACITOR-CERAMIC C7
+L conservify:CAPACITOR_CERAMIC C7
 U 1 1 560C0195
 P 6150 2300
@@
 $EndComp
 $Comp
-L fk-weather-rescue:CAPACITOR-CERAMIC C8
+L conservify:CAPACITOR_CERAMIC C8
 U 1 1 560C021E
 P 6550 2300
@@
 $EndComp
 $Comp
-L fk-weather-rescue:CAPACITOR-CERAMIC C5
+L conservify:CAPACITOR_CERAMIC C5
 U 1 1 560C02A4
 P 5750 2300
@@
 $EndComp
 $Comp
-L fk-weather-rescue:CAPACITOR-CERAMIC C4
+L conservify:CAPACITOR_CERAMIC C4
 U 1 1 560C23D4
 P 5750 3250
@@
 $EndComp
 $Comp
-L conservify:AREF #PWR013
-U 1 1 56101489
-P 1550 2700
-F 0 "#PWR013" H 1550 2550 50  0001 C CNN
-F 1 "AREF" H 1550 2840 50  0000 C CNN
-F 2 "" H 1550 2700 60  0000 C CNN
-F 3 "" H 1550 2700 60  0000 C CNN
-	1    1550 2700
-	1    0    0    -1
-$EndComp
-$Comp
-L fk-weather-rescue:CAPACITOR-CERAMIC C6
+L conservify:CAPACITOR_CERAMIC C6
 U 1 1 56101EA7
 P 1850 3050
@@
 $EndComp
 $Comp
-L fk-weather-rescue:CAPACITOR-CERAMIC C14
+L conservify:CAPACITOR_CERAMIC C14
 U 1 1 561023B1
 P 1550 3050
@@
 $EndComp
 $Comp
-L fk-weather-rescue:ATSAMD21G18A-AU U1
+L conservify:ATSAMD21G18A_AU U1
 U 1 1 56332480
 P 3900 3650
@@
 $EndComp
 $Comp
-L fk-weather-rescue:MICRO-USB J1
+L conservify:MICRO_USB J1
 U 1 1 5979086D
 P 4200 6900
@@
 $EndComp
 $Comp
-L fk-weather-rescue:CAPACITOR-CERAMIC C10
+L conservify:CAPACITOR_CERAMIC C10
 U 1 1 59790E57
 P 5000 7450
@@
 $EndComp
 $Comp
-L fk-weather-rescue:CAPACITOR-CERAMIC C9
+L conservify:CAPACITOR_CERAMIC C9
 U 1 1 59791381
 P 800 6900
@@
 $EndComp
 $Comp
-L fk-weather-rescue:CAPACITOR-CERAMIC C12
+L conservify:CAPACITOR_CERAMIC C12
 U 1 1 59792065
 P 6950 6700
@@
 $EndComp
 $Comp
-L fk-weather-rescue:CAPACITOR-CERAMIC C11
+L conservify:CAPACITOR_CERAMIC C11
 U 1 1 59792142
 P 5650 6700
@@
 $EndComp
 $Comp
-L fk-weather-rescue:LED-SINGLE D5
+L conservify:LED_SINGLE D5
 U 1 1 59BC28FF
 P 8050 3500
@@
 $EndComp
 $Comp
-L fk-weather-rescue:MOSFET-N Q4
+L conservify:MOSFET_N Q4
 U 1 1 59BC2907
 P 8950 3150
@@
 $EndComp
 $Comp
-L fk-weather-rescue:CAPACITOR-CERAMIC C18
+L conservify:CAPACITOR_CERAMIC C18
 U 1 1 5A1CAC3A
 P 6750 9100
@@
 $EndComp
 $Comp
-L fk-weather-rescue:Conn_01x06 J11
+L conservify:CONN_01x06 J11
 U 1 1 5A44A535
 P 12600 4900
@@
 $EndComp
 $Comp
-L fk-weather-rescue:Conn_01x06 J10
+L conservify:CONN_01x06 J10
 U 1 1 5A46F26B
 P 12950 2050
@@
 $EndComp
 $Comp
-L fk-weather-rescue:Conn_01x05 J2
+L conservify:CONN_01x05 J2
 U 1 1 5B3C0765
 P 8700 5850
@@
 $EndComp
 $Comp
-L fk-weather-rescue:Conn_01x04 J4
+L conservify:CONN_01x04 J4
 U 1 1 5B3C5AFF
 P 9500 5850
@@
 $EndComp
 $Comp
-L fk-weather-rescue:CAPACITOR-CERAMIC C13
+L conservify:CAPACITOR_CERAMIC C13
 U 1 1 5B3F4664
 P 11800 8550
@@
 $EndComp
 $Comp
-L fk-weather-rescue:CAPACITOR-CERAMIC C15
+L conservify:CAPACITOR_CERAMIC C15
 U 1 1 5B3F4F66
 P 15200 8650
@@
 $EndComp
 $Comp
-L fk-weather-rescue:CAPACITOR-CERAMIC C16
+L conservify:CAPACITOR_CERAMIC C16
 U 1 1 5B3F510A
 P 15600 8600
@@
 $EndComp
 $Comp
-L fk-weather-rescue:Conn_01x02 J5
+L conservify:CONN_01x02 J5
 U 1 1 5B3F92E3
 P 12900 7850
@@
 $EndComp
 $Comp
-L fk-weather-rescue:CAPACITOR-CERAMIC C17
+L conservify:CAPACITOR_CERAMIC C17
 U 1 1 5B56FA30
 P 3100 9400
@@
 $EndComp
 $Comp
-L fk-weather-rescue:CAPACITOR-CERAMIC C19
+L conservify:CAPACITOR_CERAMIC C19
 U 1 1 5B56FB8C
 P 3950 9400
@@
 $EndComp
 $Comp
-L fk-weather-rescue:Conn_01x05 J7
+L conservify:CONN_01x05 J7
 U 1 1 5B565BC0
 P 7950 5850
@@
 	7050 9800 7050 9100
 Wire Wire Line
-	1550 2700 1550 2800
-Wire Wire Line
 	1850 2800 1850 2900
 Wire Wire Line
@@
 Connection ~ 14400 1950
 Connection ~ 14400 2800
-Connection ~ 1550 2800
 Connection ~ 1850 2800
 Connection ~ 15600 8900
@@
 NoConn ~ 2550 9300
 NoConn ~ 7750 5850
+NoConn ~ 2250 3000
+NoConn ~ 2250 2700
+NoConn ~ 2250 3200
+NoConn ~ 2250 3500
+NoConn ~ 2250 3600
+NoConn ~ 2250 3800
+NoConn ~ 2250 3900
+NoConn ~ 3050 4100
+NoConn ~ 2250 4400
+NoConn ~ 2250 4600
+NoConn ~ 5350 4200
+NoConn ~ 5350 3700
+NoConn ~ 5350 3500
+$Comp
+L conservify:5V0 #PWR0101
+U 1 1 5BBDF471
+P 1150 7700
+F 0 "#PWR0101" H 1150 7550 50  0001 C CNN
+F 1 "5V0" H 1150 7840 50  0000 C CNN
+F 2 "" H 1150 7700 60  0000 C CNN
+F 3 "" H 1150 7700 60  0000 C CNN
+	1    1150 7700
+	1    0    0    -1
+$EndComp
+$Comp
+L conservify:PWR_FLAG #FLG0101
+U 1 1 5BBDF693
+P 1150 7850
+F 0 "#FLG0101" H 1150 7925 50  0001 C CNN
+F 1 "PWR_FLAG" H 1150 8023 50  0000 C CNN
+F 2 "" H 1150 7850 50  0001 C CNN
+F 3 "~" H 1150 7850 50  0001 C CNN
+	1    1150 7850
+	-1   0    0    1
+$EndComp
+Wire Wire Line
+	1150 7700 1150 7850
+$Comp
+L conservify:PWR_FLAG #FLG0102
+U 1 1 5BBDF7C1
+P 1550 7850
+F 0 "#FLG0102" H 1550 7925 50  0001 C CNN
+F 1 "PWR_FLAG" H 1550 8023 50  0000 C CNN
+F 2 "" H 1550 7850 50  0001 C CNN
+F 3 "~" H 1550 7850 50  0001 C CNN
+	1    1550 7850
+	-1   0    0    1
+$EndComp
+$Comp
+L conservify:GND #PWR0102
+U 1 1 5BC38690
+P 1550 7650
+F 0 "#PWR0102" H 1550 7400 50  0001 C CNN
+F 1 "GND" H 1550 7500 50  0001 C CNN
+F 2 "" H 1550 7650 60  0000 C CNN
+F 3 "" H 1550 7650 60  0000 C CNN
+	1    1550 7650
+	-1   0    0    1
+$EndComp
+Wire Wire Line
+	1550 7650 1550 7850
+NoConn ~ 5350 3800
+NoConn ~ 12800 5100
+NoConn ~ 12800 4600
+NoConn ~ 13150 1750
+NoConn ~ 13150 2250
+NoConn ~ 13600 2150
+NoConn ~ 13600 1850
 $EndSCHEMATC

Commit message: Use more compatible FP for flash.
Parts:
- U4: footprint conservify:SOIC-8-N -> conservify:SOIC-8-N-WIDE
Changed lines of the file:
@@
 F 0 "U4" H 5550 9550 60  0000 C CNN
 F 1 "S25FL116K0XMFI041" H 5550 8950 60  0000 C CNN
-F 2 "conservify:SOIC-8-N" H 5550 8850 60  0001 C CNN
+F 2 "conservify:SOIC-8-N-WIDE" H 5550 8850 60  0001 C CNN
 F 3 "" H 5350 9300 60  0000 C CNN
 F 4 " " H 5550 9650 50  0001 C CNN "Critical"
